Commit message: Sucessfully make controller-- need a script to sub to real hand message

File: src/urdf_display/urdf/01-myfirst.urdf (robot description, URDF)
Before this commit: robot myfirst, 1 links, 0 joints
Links:
- added link world
- link base_link: mass None -> 0.1; geometry visual cylinder length=6.0 radius=2.0
Joints:
- added joint fixed: type fixed, parent world, child base_link
