Commit message: Working URDF with model of reflex hand

File: src/urdf_display/urdf/02-myfirst_hand.urdf (robot description, URDF)
Before this commit: robot myfirst_hand, 12 links, 11 joints
Links:
- link base_link: geometry visual mesh filename=package://urdf_display/meshes/base_link.STL
- link finger_1_1: geometry visual mesh filename=package://urdf_display/meshes/swivel_1.STL
- link finger_1_2: geometry visual mesh filename=package://urdf_display/meshes/proximal_1.STL
- link finger_1_3: geometry visual mesh filename=package://urdf_display/meshes/distal_1.STL
- link finger_2_1: geometry visual mesh filename=package://urdf_display/meshes/swivel_1.STL
- link finger_2_2: geometry visual mesh filename=package://urdf_display/meshes/proximal_1.STL
- link finger_2_3: geometry visual mesh filename=package://urdf_display/meshes/distal_1.STL
- link finger_3_1: geometry visual mesh filename=package://urdf_display/meshes/swivel_1.STL
- link finger_3_2: geometry visual mesh filename=package://urdf_display/meshes/proximal_1.STL
- link finger_3_3: geometry visual mesh filename=package://urdf_display/meshes/distal_1.STL
- link sub_base_link: geometry visual cylinder length=0.2 radius=0.5
Joints:
- joint base_to_finger_1_1: axis 0 0 1 -> 0 0 -1; origin xyz=1 1.25 0.75 -> xyz=0.0503973683071414 -0.026 0.063 rpy=6.75550818663469E-16 1.97993848419069E-16 -2.77555756156289E-16
- joint base_to_finger_2_1: axis 0 0 1 -> 0 0 -1; origin xyz=-1 1.25 0.75 -> xyz=0.0503973683071413 0.0259999999999999 0.063 rpy=1.22459340959228E-15 -7.33448407631817E-16 -1.66533453693773E-16
- joint base_to_finger_3_1: axis 0 0 1 -> 0 0 -1; origin xyz=0 -1.25 0.75 -> xyz=0 0 0 rpy=0 0 0
- joint finger_1_1_to_finger_1_2: axis 1 0 0 -> 0 -1 0; origin xyz=0 0 0.5 -> xyz=0.01 0 0.0186 rpy=-6.20039667432211E-16 0.28 2.22044604925031E-16
- joint finger_1_2_to_finger_1_3: axis 1 0 0 -> 0 -1 0; origin xyz=0 2 0 -> xyz=0.07600000000000001 0 0.00250000000000002 rpy=0 0 0
- joint finger_2_1_to_finger_2_2: axis 1 0 0 -> 0 -1 0; origin xyz=0 0 0.5 -> xyz=0.01 0 0.0186 rpy=-1.16908225836102E-15 0.28 1.11022302462515E-16
- joint finger_2_2_to_finger_2_3: axis 1 0 0 -> 0 -1 0; origin xyz=0 2 0 -> xyz=0.0760000000000001 0 0.00249999999999997 rpy=0 0 0
- joint finger_3_1_to_finger_3_2: axis -1 0 0 -> 0 -1 0; origin xyz=0 0 0.5 -> xyz=-0.0299999999999996 0 0.0816000000000002 rpy=-5.55111512312578E-17 0.28 3.14159265358979
- joint finger_3_2_to_finger_3_3: axis -1 0 0 -> 0 -1 0; origin xyz=0 -2 0 -> xyz=0.0760000000000001 0 0.0025 rpy=-1.48887961834512E-45 -1.0995850059156E-76 -7.38531841236285E-32
